File: schematics/playground1/pic32.kicad_sch (KiCad schematic)
At the start: 1 part, among them U4 PIC32MX250F128B_I_SS

Commit message: first draft of pic32 schematic complete
Parts:
- added C1, C2: 18pF, symbol Device:C
- added C3: 10uF, symbol Device:C
- added D1: LED, symbol Device:LED
- added R1, R3: 470K, symbol Device:R
- added R2: 1K, symbol Device:R
- added SW1, SW2: SW_Push, symbol Switch:SW_Push
- added Y1: 8MHz, symbol Device:Crystal
Connections:
- net AGND: now also C1.1, C2.2, C3.2, R2.1, R3.2, SW2.1
- net DVDD_3V3: now also R1.1, SW1.1
- net at U4.1 (MCLR): now also R1.2, SW2.2
- net at U4.10 (OSC2/CLKO/RPA3/PMA0/RA3): now also C2.1, Y1.1
- net at U4.11 (SOSCI/RPB4/RB4): now also R3.1, SW1.2
- net at U4.20 (VCAP): now also C3.1
- net at U4.4 (PGED1/AN2/C1IND/C2INB/C3IND/RPB0/PMD0/RB0): now also D1.2 (A)
- net at U4.9 (OSC1/CLKI/RPA2/RA2): now also C1.2, Y1.2
- new net: D1.1 (K), R2.2

Commit message: update voltage regulators to ones we can buy
Parts:
- renumbered C3 to C?, C2 to C?, C1 to C?, D1 to D?, R2 to R?, R1 to R?, R3 to R?, SW2 to SW?, SW1 to SW?, Y1 to Y?
Changed lines of the file:
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@@
 		(dnp no)
 		(fields_autoplaced yes)
-		(property "Reference" "C3"
+		(property "Reference" "C?"
 			(at 227.33 82.55 90)
 			(effects
@@
 		)
 		(instances
+			(project "playground"
+				(path "/238de170-6a90-40ad-afaf-ab931b754487/6c9dea1e-c151-4e07-9538-ad97d255bf92"
+					(reference "C?")
+					(unit 1)
+				)
+			)
 			(project ""
 				(path "/7c95cdee-8526-4ace-82fb-b64957eb01de"
@@
 		(dnp no)
 		(fields_autoplaced yes)
-		(property "Reference" "D1"
+		(property "Reference" "D?"
 			(at 49.2125 71.12 0)
 			(effects
@@
 		(dnp no)
 		(fields_autoplaced yes)
-		(property "Reference" "U?"
+		(property "Reference" "U4"
 			(at 133.35 59.69 0)
 			(effects
@@
 		(dnp no)
 		(fields_autoplaced yes)
-		(property "Reference" "SW2"
+		(property "Reference" "SW?"
 			(at 27.94 59.69 0)
 			(effects
@@
 		)
 		(instances
+			(project "playground"
+				(path "/238de170-6a90-40ad-afaf-ab931b754487/6c9dea1e-c151-4e07-9538-ad97d255bf92"
+					(reference "SW?")
+					(unit 1)
+				)
+			)
 			(project ""
 				(path "/7c95cdee-8526-4ace-82fb-b64957eb01de"
@@
 		(dnp no)
 		(fields_autoplaced yes)
-		(property "Reference" "SW1"
+		(property "Reference" "SW?"
 			(at 35.56 99.06 0)
 			(effects
@@
 		)
 		(instances
+			(project "playground"
+				(path "/238de170-6a90-40ad-afaf-ab931b754487/6c9dea1e-c151-4e07-9538-ad97d255bf92"
+					(reference "SW?")
+					(unit 1)
+				)
+			)
 			(project ""
 				(path "/7c95cdee-8526-4ace-82fb-b64957eb01de"
@@
 		(dnp no)
 		(fields_autoplaced yes)
-		(property "Reference" "C2"
+		(property "Reference" "C?"
 			(at 26.67 90.17 90)
 			(effects
@@
 		)
 		(instances
+			(project "playground"
+				(path "/238de170-6a90-40ad-afaf-ab931b754487/6c9dea1e-c151-4e07-9538-ad97d255bf92"
+					(reference "C?")
+					(unit 1)
+				)
+			)
 			(project ""
 				(path "/7c95cdee-8526-4ace-82fb-b64957eb01de"
@@
 		(dnp no)
 		(fields_autoplaced yes)
-		(property "Reference" "C1"
+		(property "Reference" "C?"
 			(at 26.67 76.2 90)
 			(effects
@@
 		)
 		(instances
+			(project "playground"
+				(path "/238de170-6a90-40ad-afaf-ab931b754487/6c9dea1e-c151-4e07-9538-ad97d255bf92"
+					(reference "C?")
+					(unit 1)
+				)
+			)
 			(project ""
 				(path "/7c95cdee-8526-4ace-82fb-b64957eb01de"
@@
 		(dnp no)
 		(fields_autoplaced yes)
-		(property "Reference" "Y1"
+		(property "Reference" "Y?"
 			(at 44.45 90.1699 90)
 			(effects
@@
 		)
 		(instances
+			(project "playground"
+				(path "/238de170-6a90-40ad-afaf-ab931b754487/6c9dea1e-c151-4e07-9538-ad97d255bf92"
+					(reference "Y?")
+					(unit 1)
+				)
+			)
 			(project ""
 				(path "/7c95cdee-8526-4ace-82fb-b64957eb01de"
@@
 		(dnp no)
 		(fields_autoplaced yes)
-		(property "Reference" "R2"
+		(property "Reference" "R?"
 			(at 43.18 71.12 90)
 			(effects
@@
 		(dnp no)
 		(fields_autoplaced yes)
-		(property "Reference" "R1"
+		(property "Reference" "R?"
 			(at 54.61 57.15 90)
 			(effects
@@
 		(dnp no)
 		(fields_autoplaced yes)
-		(property "Reference" "R3"
+		(property "Reference" "R?"
 			(at 44.45 109.2199 0)
 			(effects
@@
 		)
 		(instances
-			(project ""
-				(path "/7c95cdee-8526-4ace-82fb-b64957eb01de"
+			(project "playground"
+				(path "/238de170-6a90-40ad-afaf-ab931b754487/6c9dea1e-c151-4e07-9538-ad97d255bf92"
+					(reference "R?")
+					(unit 1)
+				)
+			)
+			(project ""
+				(path "/7c95cdee-8526-4ace-82fb-b64957eb01de"
